Commit message: Fixed mimic joints and set correct joint limits
 - Mimic joints work as intended, but xacro is a bit of a pain for
 "optional" blocks (e.g. some revolute joints don't mimic others)
 - Joint min/max limits are set correctly, 0.0 position is default
 - Add mesh_roll as the eye_right mesh is 0.01 radians off

File: marty2_description/urdf/marty2/marty2_structure.xacro (robot description, xacro)
@@ -18,25 +18,36 @@
   <xacro:revolute name="eye_left" parent="head" material="white" mesh="eye_left" rot_r="1">
     <origin xyz="0.04570 0.02410 0.04671" rpy="0 0 0"/>
+    <mimic joint="eye_left_joint" multiplier="0"/> <!-- Not mimicking -->
+    <limit effort="30" velocity="1.0" lower="-3.0" upper="0.25" />
   </xacro:revolute>
-  <xacro:revolute name="eye_right" parent="head" material="white" mesh="eye_right" rot_r="1">
+  <xacro:revolute name="eye_right" parent="head" material="white" mesh="eye_right" mesh_roll="0.01" rot_r="1">
     <origin xyz="0.04570 -0.02410 0.04671" rpy="0 0 0"/>
+    <mimic joint="eye_left_joint" multiplier="-1"/>
+    <limit effort="30" velocity="1.0" lower="-0.25" upper="3.0" />
   </xacro:revolute>
-  <!-- Arms -->
+  <!-- Left arm -->
   <xacro:revolute name="arm_servo_gear_left" parent="side_panel_left" material="yellow" mesh_pitch="-0.5585" mesh="arm_servo_gear" rot_p="1">
     <origin xyz="0 0.00025 0" rpy="0 0 0"/>
-    <!-- <mimic joint="arm_servo_gear_left_joint" multiplier="0"/> -->
-  </xacro:revolute>
-  <xacro:revolute name="arm_servo_gear_right" parent="side_panel_right" material="yellow" mesh="arm_servo_gear" mesh_pitch="-0.5585" mesh_yaw="3.1416" rot_p="1">
-    <origin xyz="0 -0.00025 0" rpy="0 0 0"/>
-    <!-- <mimic joint="arm_servo_gear_right_joint" multiplier="0"/> -->
+    <mimic joint="arm_servo_gear_left_joint" multiplier="0"/> <!-- Not Mimicking -->
+    <limit effort="30" velocity="1.0" lower="-0.95" upper="2.05" />
   </xacro:revolute>
   <xacro:revolute name="arm_left" parent="side_panel_left" material="yellow" mesh="arm" rot_p="1">
     <origin xyz="0 0 -0.03020" rpy="0 0 0"/>
+    <mimic joint="arm_servo_gear_left_joint" multiplier="-1.307692308"/>
+    <limit effort="30" velocity="1.0" lower="-2.68" upper="1.24" />
   </xacro:revolute>
   <xacro:fixed name="hand_left" parent="arm_left" material="yellow" mesh="hand">
     <origin xyz="0.00000 0.0330 -0.05539" rpy="0.3490658504 0 0"/>
   </xacro:fixed>
+  <!-- Right arm -->
+  <xacro:revolute name="arm_servo_gear_right" parent="side_panel_right" material="yellow" mesh="arm_servo_gear" mesh_pitch="0.5585" mesh_yaw="3.1416" rot_p="1">
+    <origin xyz="0 -0.00025 0" rpy="0 0 0"/>
+    <mimic joint="arm_servo_gear_right_joint" multiplier="0"/> <!-- Not mimicking -->
+    <limit effort="30" velocity="1.0" lower="-0.95" upper="2.05" />
+  </xacro:revolute>
   <xacro:revolute name="arm_right" parent="side_panel_right" material="yellow" mesh="arm" mesh_yaw="3.1416" rot_p="1">
     <origin xyz="0 0 -0.03020" rpy="0 0 0"/>
+    <mimic joint="arm_servo_gear_right_joint" multiplier="-1.307692308"/>
+    <limit effort="30" velocity="1.0" lower="-2.68" upper="1.24" />
   </xacro:revolute>
   <xacro:fixed name="hand_right" parent="arm_right" material="yellow" mesh="hand">

File: marty2_description/urdf/revolute.xacro (robot description, xacro)
@@ -1,5 +1,5 @@
 <?xml version="1.0"?>
 <robot xmlns:xacro="http://www.ros.org/wiki/xacro">
-  <xacro:macro name="revolute" params="name parent material mesh mesh_pitch:=0 mesh_yaw:=0 rot_r:=0 rot_p:=0 rot_y:=0 *origin">
+  <xacro:macro name="revolute" params="name parent material mesh mesh_roll:=0 mesh_pitch:=0 mesh_yaw:=0 rot_r:=0 rot_p:=0 rot_y:=0 *origin *mimic *limit">
     <joint name="${name}_joint" type="revolute">
       <xacro:insert_block name="origin"/>
@@ -7,5 +7,6 @@
       <child link="${name}"/>
       <axis xyz="${rot_r} ${rot_p} ${rot_y}"/>
-      <limit effort="30" velocity="1.0" lower="-1.0" upper="1.0" />
+      <xacro:insert_block name="mimic"/>
+      <xacro:insert_block name="limit"/>
     </joint>
     <link name="${name}">
@@ -19,5 +20,5 @@
           <mesh filename="http://0.0.0.0:8000/${mesh}.stl"/>
         </geometry>
-        <origin xyz="0 0 0" rpy="0 ${mesh_pitch} ${mesh_yaw}"/>
+        <origin xyz="0 0 0" rpy="${mesh_roll} ${mesh_pitch} ${mesh_yaw}"/>
         <material name="${material}"/>
       </visual>
@@ -26,5 +27,5 @@
           <mesh filename="http://0.0.0.0:8000/${mesh}.stl"/>
         </geometry>
-        <origin xyz="0 0 0" rpy="0 ${mesh_pitch} ${mesh_yaw}"/>
+        <origin xyz="0 0 0" rpy="${mesh_roll} ${mesh_pitch} ${mesh_yaw}"/>
         <material name="${material}"/>
       </collision>
