Commit message: Setup ROS2 Control interface and add all joints
 - Implement Joint Trajectory Position Controller for active joints
 - Implement mimicking of passive joints following active joints
 - Add demo trajectory commands launch file to send control commands
 - Update xacro files to keep things modular and semi-sane

File: marty2_description/urdf/marty2/marty2.xacro (robot description, xacro)
@@ -7,3 +7,5 @@
   <!-- Bolt-on sensors go here -->
   <!-- <xacro:include filename="$(find marty2_description)/urdf/marty2/marty2_sensors.xacro"/> -->
+  <xacro:include filename="$(find marty2_description)/ros2_control/marty2.ros2_control.xacro" />
+  <xacro:marty2_ros2_control name="marty2"/>
 </robot>

File: marty2_description/urdf/marty2/marty2_structure.xacro (robot description, xacro)
@@ -18,22 +18,18 @@
   <xacro:revolute name="eye_left" parent="head" material="white" mesh="eye_left" rot_r="1">
     <origin xyz="0.04570 0.02410 0.04671" rpy="0 0 0"/>
-    <mimic joint="eye_left_joint" multiplier="0"/> <!-- Not mimicking -->
-    <limit effort="30" velocity="1.0" lower="-3.0" upper="0.25" />
+    <limit effort="30" velocity="6.29" lower="-3.0" upper="0.25" />
   </xacro:revolute>
-  <xacro:revolute name="eye_right" parent="head" material="white" mesh="eye_right" mesh_roll="0.01" rot_r="1">
+  <xacro:revolute name="eye_right" parent="head" material="white" mesh="eye_right" mesh_roll="0.01" rot_r="1" mimic_joint="eye_left_joint" mimic_mult="-1">
     <origin xyz="0.04570 -0.02410 0.04671" rpy="0 0 0"/>
-    <mimic joint="eye_left_joint" multiplier="-1"/>
-    <limit effort="30" velocity="1.0" lower="-0.25" upper="3.0" />
+    <limit effort="30" velocity="6.29" lower="-0.25" upper="3.0" />
   </xacro:revolute>
   <!-- Left arm -->
   <xacro:revolute name="arm_servo_gear_left" parent="side_panel_left" material="yellow" mesh_pitch="-0.5585" mesh="arm_servo_gear" rot_p="1">
     <origin xyz="0 0.00025 0" rpy="0 0 0"/>
-    <mimic joint="arm_servo_gear_left_joint" multiplier="0"/> <!-- Not Mimicking -->
-    <limit effort="30" velocity="1.0" lower="-0.95" upper="2.05" />
+    <limit effort="30" velocity="6.29" lower="-0.95" upper="2.05" />
   </xacro:revolute>
-  <xacro:revolute name="arm_left" parent="side_panel_left" material="yellow" mesh="arm" rot_p="1">
+  <xacro:revolute name="arm_left" parent="side_panel_left" material="yellow" mesh="arm" rot_p="1" mimic_joint="arm_servo_gear_left_joint" mimic_mult="-1.307692308">
     <origin xyz="0 0 -0.03020" rpy="0 0 0"/>
-    <mimic joint="arm_servo_gear_left_joint" multiplier="-1.307692308"/>
-    <limit effort="30" velocity="1.0" lower="-2.68" upper="1.24" />
+    <limit effort="30" velocity="6.29" lower="-2.68" upper="1.24" />
   </xacro:revolute>
   <xacro:fixed name="hand_left" parent="arm_left" material="yellow" mesh="hand">
@@ -43,21 +39,88 @@
   <xacro:revolute name="arm_servo_gear_right" parent="side_panel_right" material="yellow" mesh="arm_servo_gear" mesh_pitch="0.5585" mesh_yaw="3.1416" rot_p="1">
     <origin xyz="0 -0.00025 0" rpy="0 0 0"/>
-    <mimic joint="arm_servo_gear_right_joint" multiplier="0"/> <!-- Not mimicking -->
-    <limit effort="30" velocity="1.0" lower="-0.95" upper="2.05" />
+    <limit effort="30" velocity="6.29" lower="-0.95" upper="2.05" />
   </xacro:revolute>
-  <xacro:revolute name="arm_right" parent="side_panel_right" material="yellow" mesh="arm" mesh_yaw="3.1416" rot_p="1">
+  <xacro:revolute name="arm_right" parent="side_panel_right" material="yellow" mesh="arm" mesh_yaw="3.1416" rot_p="1" mimic_joint="arm_servo_gear_right_joint" mimic_mult="-1.307692308">
     <origin xyz="0 0 -0.03020" rpy="0 0 0"/>
-    <mimic joint="arm_servo_gear_right_joint" multiplier="-1.307692308"/>
-    <limit effort="30" velocity="1.0" lower="-2.68" upper="1.24" />
+    <limit effort="30" velocity="6.29" lower="-2.68" upper="1.24" />
   </xacro:revolute>
   <xacro:fixed name="hand_right" parent="arm_right" material="yellow" mesh="hand">
     <origin xyz="0.00000 -0.0330 -0.05539" rpy="-0.3490658504 0 0"/>
   </xacro:fixed>
-  <!-- Legs -->
+  <!-- Left leg -->
   <xacro:fixed name="hip_left" parent="head" material="blue" mesh="hip">
     <origin xyz="0.01087 0.04709 -0.01465" rpy="0.0000 0.0000 0.0000"/>
   </xacro:fixed>
+  <xacro:revolute name="leg_left_thigh_front" parent="hip_left" material="blue" mesh="thigh" rot_p="1">
+    <origin xyz="0.00000  0.00025 0.00000" rpy="0.0000 0.0000 0.0000"/>
+    <limit effort="30" velocity="6.29" lower="-1.0" upper="1.0" />
+  </xacro:revolute>
+  <xacro:revolute name="leg_left_thigh_back" parent="hip_left" material="blue" mesh="thigh" mesh_yaw="3.1416" mimic_joint="leg_left_thigh_front_joint" mimic_mult="1" rot_p="1">
+    <origin xyz="-0.01620 -0.03795  0.00000" rpy="0.0000 0.0000 0.0000"/>
+    <limit effort="30" velocity="6.29" lower="-1.0" upper="1.0" />
+  </xacro:revolute>
+  <xacro:revolute name="leg_left_knee_upper" parent="leg_left_thigh_front" material="blue" mesh="knee_upper" mimic_joint="leg_left_thigh_front_joint" mimic_mult="-1" rot_p="1">
+    <origin xyz="0.00000  -0.00015  -0.05000" rpy="0.0000 0.0000 0.0000"/>
+    <limit effort="30" velocity="6.29" lower="-1.0" upper="1.0" />
+  </xacro:revolute>
+  <xacro:fixed name="leg_left_twist_upper" parent="leg_left_knee_upper" material="yellow" mesh="twist_upper">
+    <origin xyz="-0.00810 -0.01885  -0.00968" rpy="0.0000 0.0000 0.0000"/>
+  </xacro:fixed>
+  <xacro:revolute name="leg_left_twist_lower" parent="leg_left_twist_upper" material="yellow" mesh="twist_lower" rot_y="1">
+    <origin xyz="0.0000 0.0000 0.0000" rpy="0.0000 0.0000 0.0000"/>
+    <limit effort="30" velocity="6.29" lower="-1.0" upper="1.0" />
+  </xacro:revolute>
+  <xacro:fixed name="leg_left_knee_lower" parent="leg_left_twist_lower" material="blue" mesh="knee_lower">
+    <origin xyz="-0.01885 0.00810 -0.02075" rpy="0.0000 0.0000 0.0000"/>
+  </xacro:fixed>
+  <xacro:revolute name="leg_left_shin_exterior" parent="leg_left_knee_lower" material="blue" mesh="shin" rot_r="1">
+    <origin xyz="0.0000 0.0000 0.0000" rpy="0.0000 0.0000 0.0000"/>
+    <limit effort="30" velocity="6.29" lower="-1.0" upper="1.0" />
+  </xacro:revolute>
+  <xacro:revolute name="leg_left_shin_interior" parent="leg_left_knee_lower" material="blue" mesh="shin" mesh_yaw="3.1416" mimic_joint="leg_left_shin_exterior_joint" mimic_mult="1" rot_r="1">
+    <origin xyz="0.03770  -0.01620  0.00000" rpy="0.0000 0.0000 0.0000"/>
+    <limit effort="30" velocity="6.29" lower="-1.0" upper="1.0" />
+  </xacro:revolute>
+  <xacro:revolute name="foot_left" parent="leg_left_shin_exterior" material="yellow" mesh="foot" mimic_joint="leg_left_shin_exterior_joint" mimic_mult="-1" rot_r="1">
+    <origin xyz="0.00000  0.00000 -0.05000" rpy="0.0000 0.0000 0.0000"/>
+    <limit effort="30" velocity="6.29" lower="-1.0" upper="1.0" />
+  </xacro:revolute>
+  <!-- Right leg -->
   <xacro:fixed name="hip_right" parent="head" material="blue" mesh="hip">
     <origin xyz="0.01087 -0.00941 -0.01465" rpy="0.0000 0.0000 0.0000"/>
   </xacro:fixed>
+  <xacro:revolute name="leg_right_thigh_front" parent="hip_right" material="blue" mesh="thigh" rot_p="1">
+    <origin xyz="0.00000  0.00025 0.00000" rpy="0.0000 0.0000 0.0000"/>
+    <limit effort="30" velocity="6.29" lower="-1.0" upper="1.0" />
+  </xacro:revolute>
+  <xacro:revolute name="leg_right_thigh_back" parent="hip_right" material="blue" mesh="thigh" mesh_yaw="3.1416" mimic_joint="leg_right_thigh_front_joint" mimic_mult="1" rot_p="1">
+    <origin xyz="-0.01620 -0.03795  0.00000" rpy="0.0000 0.0000 0.0000"/>
+    <limit effort="30" velocity="6.29" lower="-1.0" upper="1.0" />
+  </xacro:revolute>
+  <xacro:revolute name="leg_right_knee_upper" parent="leg_right_thigh_front" material="blue" mesh="knee_upper" mimic_joint="leg_right_thigh_front_joint" mimic_mult="-1" rot_p="1">
+    <origin xyz="0.00000  -0.00015  -0.05000" rpy="0.0000 0.0000 0.0000"/>
+    <limit effort="30" velocity="6.29" lower="-1.0" upper="1.0" />
+  </xacro:revolute>
+  <xacro:fixed name="leg_right_twist_upper" parent="leg_right_knee_upper" material="yellow" mesh="twist_upper">
+    <origin xyz="-0.00810 -0.01885  -0.00968" rpy="0.0000 0.0000 0.0000"/>
+  </xacro:fixed>
+  <xacro:revolute name="leg_right_twist_lower" parent="leg_right_twist_upper" material="yellow" mesh="twist_lower" rot_y="1">
+    <origin xyz="0.0000 0.0000 0.0000" rpy="0.0000 0.0000 0.0000"/>
+    <limit effort="30" velocity="6.29" lower="-1.0" upper="1.0" />
+  </xacro:revolute>
+  <xacro:fixed name="leg_right_knee_lower" parent="leg_right_twist_lower" material="blue" mesh="knee_lower">
+    <origin xyz="-0.01885 0.00810 -0.02075" rpy="0.0000 0.0000 0.0000"/>
+  </xacro:fixed>
+  <xacro:revolute name="leg_right_shin_exterior" parent="leg_right_knee_lower" material="blue" mesh="shin" mesh_yaw="3.1416" mimic_joint="leg_right_shin_interior_joint" mimic_mult="1" rot_r="1">
+    <origin xyz="0.03770  -0.01620  0.00000" rpy="0.0000 0.0000 0.0000"/>
+    <limit effort="30" velocity="6.29" lower="-1.0" upper="1.0" />
+  </xacro:revolute>
+  <xacro:revolute name="leg_right_shin_interior" parent="leg_right_knee_lower" material="blue" mesh="shin" rot_r="1">
+    <origin xyz="0.0000 0.0000 0.0000" rpy="0.0000 0.0000 0.0000"/>
+    <limit effort="30" velocity="6.29" lower="-1.0" upper="1.0" />
+  </xacro:revolute>
+  <xacro:revolute name="foot_right" parent="leg_right_shin_interior" material="yellow" mesh="foot" mesh_x="0.03790" mesh_y="-0.01620" mesh_yaw="3.1416" mimic_joint="leg_right_shin_interior_joint" mimic_mult="-1" rot_r="1">
+    <origin xyz="0 0 -0.05000" rpy="0.0000 0.0000 0.0000"/>
+    <limit effort="30" velocity="6.29" lower="-1.0" upper="1.0" />
+  </xacro:revolute>
 </robot>

File: marty2_description/urdf/revolute.xacro (robot description, xacro)
@@ -1,5 +1,5 @@
 <?xml version="1.0"?>
 <robot xmlns:xacro="http://www.ros.org/wiki/xacro">
-  <xacro:macro name="revolute" params="name parent material mesh mesh_roll:=0 mesh_pitch:=0 mesh_yaw:=0 rot_r:=0 rot_p:=0 rot_y:=0 *origin *mimic *limit">
+  <xacro:macro name="revolute" params="name parent material mesh mesh_x:=0 mesh_y:=0 mesh_roll:=0 mesh_pitch:=0 mesh_yaw:=0 rot_r:=0 rot_p:=0 rot_y:=0 mimic_joint:='' mimic_mult:='' *origin *limit">
     <joint name="${name}_joint" type="revolute">
       <xacro:insert_block name="origin"/>
@@ -7,6 +7,8 @@
       <child link="${name}"/>
       <axis xyz="${rot_r} ${rot_p} ${rot_y}"/>
-      <xacro:insert_block name="mimic"/>
-      <xacro:insert_block name="limit"/>
+      <xacro:if value="${mimic_joint != ''}">
+        <mimic joint="${mimic_joint}" multiplier="${mimic_mult}"/>
+      </xacro:if>
+      <xacro:insert_block name="limit" />
     </joint>
     <link name="${name}">
@@ -20,5 +22,5 @@
           <mesh filename="http://0.0.0.0:8000/${mesh}.stl"/>
         </geometry>
-        <origin xyz="0 0 0" rpy="${mesh_roll} ${mesh_pitch} ${mesh_yaw}"/>
+        <origin xyz="${mesh_x} ${mesh_y} 0" rpy="${mesh_roll} ${mesh_pitch} ${mesh_yaw}"/>
         <material name="${material}"/>
       </visual>
@@ -27,5 +29,5 @@
           <mesh filename="http://0.0.0.0:8000/${mesh}.stl"/>
         </geometry>
-        <origin xyz="0 0 0" rpy="${mesh_roll} ${mesh_pitch} ${mesh_yaw}"/>
+        <origin xyz="${mesh_x} ${mesh_y} 0" rpy="${mesh_roll} ${mesh_pitch} ${mesh_yaw}"/>
         <material name="${material}"/>
       </collision>
