Commit message: Update Readme with gif to demonstrate walk loop
 - Walk loop positions provided in demo .yaml file
 - Also fix .urdf file with actual package path

File: marty2_description/urdf/marty2/marty2.urdf (robot description, URDF)
Before this commit: robot marty2, 32 links, 31 joints
Links:
- link arm_left: geometry collision mesh filename=package://marty2_description/meshes/arm.stl; visual mesh filename=package://marty2_description/meshes/arm.stl
- link arm_right: geometry collision mesh filename=package://marty2_description/meshes/arm.stl; visual mesh filename=package://marty2_description/meshes/arm.stl
- link arm_servo_gear_left: geometry collision mesh filename=package://marty2_description/meshes/arm_servo_gear.stl; visual mesh filename=package://marty2_description/meshes/arm_servo_gear.stl
- link arm_servo_gear_right: geometry collision mesh filename=package://marty2_description/meshes/arm_servo_gear.stl; visual mesh filename=package://marty2_description/meshes/arm_servo_gear.stl
- link eye_left: geometry collision mesh filename=package://marty2_description/meshes/eye_left.stl; visual mesh filename=package://marty2_description/meshes/eye_left.stl
- link eye_right: geometry collision mesh filename=package://marty2_description/meshes/eye_right.stl; visual mesh filename=package://marty2_description/meshes/eye_right.stl
- link foot_left: geometry collision mesh filename=package://marty2_description/meshes/foot.stl; visual mesh filename=package://marty2_description/meshes/foot.stl
- link foot_right: geometry collision mesh filename=package://marty2_description/meshes/foot.stl; visual mesh filename=package://marty2_description/meshes/foot.stl
- link hand_left: geometry collision mesh filename=package://marty2_description/meshes/hand.stl; visual mesh filename=package://marty2_description/meshes/hand.stl
- link hand_right: geometry collision mesh filename=package://marty2_description/meshes/hand.stl; visual mesh filename=package://marty2_description/meshes/hand.stl
- link head: geometry collision mesh filename=package://marty2_description/meshes/head.stl; visual mesh filename=package://marty2_description/meshes/head.stl
- link hip_left: geometry collision mesh filename=package://marty2_description/meshes/hip.stl; visual mesh filename=package://marty2_description/meshes/hip.stl
- link hip_right: geometry collision mesh filename=package://marty2_description/meshes/hip.stl; visual mesh filename=package://marty2_description/meshes/hip.stl
- link leg_left_knee_lower: geometry collision mesh filename=package://marty2_description/meshes/knee_lower.stl; visual mesh filename=package://marty2_description/meshes/knee_lower.stl
- link leg_left_knee_upper: geometry collision mesh filename=package://marty2_description/meshes/knee_upper.stl; visual mesh filename=package://marty2_description/meshes/knee_upper.stl
- link leg_left_shin_exterior: geometry collision mesh filename=package://marty2_description/meshes/shin.stl; visual mesh filename=package://marty2_description/meshes/shin.stl
- link leg_left_shin_interior: geometry collision mesh filename=package://marty2_description/meshes/shin.stl; visual mesh filename=package://marty2_description/meshes/shin.stl
- link leg_left_thigh_back: geometry collision mesh filename=package://marty2_description/meshes/thigh.stl; visual mesh filename=package://marty2_description/meshes/thigh.stl
- link leg_left_thigh_front: geometry collision mesh filename=package://marty2_description/meshes/thigh.stl; visual mesh filename=package://marty2_description/meshes/thigh.stl
- link leg_left_twist_lower: geometry collision mesh filename=package://marty2_description/meshes/twist_lower.stl; visual mesh filename=package://marty2_description/meshes/twist_lower.stl
- link leg_left_twist_upper: geometry collision mesh filename=package://marty2_description/meshes/twist_upper.stl; visual mesh filename=package://marty2_description/meshes/twist_upper.stl
- link leg_right_knee_lower: geometry collision mesh filename=package://marty2_description/meshes/knee_lower.stl; visual mesh filename=package://marty2_description/meshes/knee_lower.stl
- link leg_right_knee_upper: geometry collision mesh filename=package://marty2_description/meshes/knee_upper.stl; visual mesh filename=package://marty2_description/meshes/knee_upper.stl
- link leg_right_shin_exterior: geometry collision mesh filename=package://marty2_description/meshes/shin.stl; visual mesh filename=package://marty2_description/meshes/shin.stl
- link leg_right_shin_interior: geometry collision mesh filename=package://marty2_description/meshes/shin.stl; visual mesh filename=package://marty2_description/meshes/shin.stl
- link leg_right_thigh_back: geometry collision mesh filename=package://marty2_description/meshes/thigh.stl; visual mesh filename=package://marty2_description/meshes/thigh.stl
- link leg_right_thigh_front: geometry collision mesh filename=package://marty2_description/meshes/thigh.stl; visual mesh filename=package://marty2_description/meshes/thigh.stl
- link leg_right_twist_lower: geometry collision mesh filename=package://marty2_description/meshes/twist_lower.stl; visual mesh filename=package://marty2_description/meshes/twist_lower.stl
- link leg_right_twist_upper: geometry collision mesh filename=package://marty2_description/meshes/twist_upper.stl; visual mesh filename=package://marty2_description/meshes/twist_upper.stl
- link side_panel_left: geometry collision mesh filename=package://marty2_description/meshes/side_panel.stl; visual mesh filename=package://marty2_description/meshes/side_panel.stl
- link side_panel_right: geometry collision mesh filename=package://marty2_description/meshes/side_panel.stl; visual mesh filename=package://marty2_description/meshes/side_panel.stl
Joints:
- removed joint leg_left_shin_exterior_joint
- removed joint leg_left_thigh_front_joint
- removed joint leg_left_twist_lower_joint
- removed joint leg_right_shin_interior_joint
- removed joint leg_right_thigh_front_joint
- removed joint leg_right_twist_lower_joint
- added joint leg_left_shin_joint: type revolute, parent leg_left_knee_lower, child leg_left_shin_exterior, origin xyz=0.0000 0.0000 0.0000 rpy=0.0000 0.0000 0.0000, axis 1 0 0, limit lower=-1.0 upper=1.0 effort=30 velocity=6.29
- added joint leg_left_thigh_joint: type revolute, parent hip_left, child leg_left_thigh_front, origin xyz=0.00000  0.00025 0.00000 rpy=0.0000 0.0000 0.0000, axis 0 1 0, limit lower=-1.0 upper=1.0 effort=30 velocity=6.29
- added joint leg_left_twist_joint: type revolute, parent leg_left_twist_upper, child leg_left_twist_lower, origin xyz=0.0000 0.0000 0.0000 rpy=0.0000 0.0000 0.0000, axis 0 0 1, limit lower=-1.0 upper=1.0 effort=30 velocity=6.29
- added joint leg_right_shin_joint: type revolute, parent leg_right_knee_lower, child leg_right_shin_interior, origin xyz=0.0000 0.0000 0.0000 rpy=0.0000 0.0000 0.0000, axis 1 0 0, limit lower=-1.0 upper=1.0 effort=30 velocity=6.29
- added joint leg_right_thigh_joint: type revolute, parent hip_right, child leg_right_thigh_front, origin xyz=0.00000  0.00025 0.00000 rpy=0.0000 0.0000 0.0000, axis 0 1 0, limit lower=-1.0 upper=1.0 effort=30 velocity=6.29
- added joint leg_right_twist_joint: type revolute, parent leg_right_twist_upper, child leg_right_twist_lower, origin xyz=0.0000 0.0000 0.0000 rpy=0.0000 0.0000 0.0000, axis 0 0 1, limit lower=-1.0 upper=1.0 effort=30 velocity=6.29
- joint foot_left_joint: mimic joint=leg_left_shin_exterior_joint multiplier=-1 -> joint=leg_left_shin_joint multiplier=-1
- joint foot_right_joint: mimic joint=leg_right_shin_interior_joint multiplier=-1 -> joint=leg_right_shin_joint multiplier=-1
- joint leg_left_knee_upper_joint: mimic joint=leg_left_thigh_front_joint multiplier=-1 -> joint=leg_left_thigh_joint multiplier=-1
- joint leg_left_shin_interior_joint: mimic joint=leg_left_shin_exterior_joint multiplier=1 -> joint=leg_left_shin_joint multiplier=1
- joint leg_left_thigh_back_joint: mimic joint=leg_left_thigh_front_joint multiplier=1 -> joint=leg_left_thigh_joint multiplier=1
- joint leg_right_knee_upper_joint: mimic joint=leg_right_thigh_front_joint multiplier=-1 -> joint=leg_right_thigh_joint multiplier=-1
- joint leg_right_shin_exterior_joint: mimic joint=leg_right_shin_interior_joint multiplier=1 -> joint=leg_right_shin_joint multiplier=1
- joint leg_right_thigh_back_joint: mimic joint=leg_right_thigh_front_joint multiplier=1 -> joint=leg_right_thigh_joint multiplier=1
