Commit message: Upload and setup Marty xacro structure up to hips
 - All STL files in meshes folder
 - Separate xacro files per joint type
 - Separate joint name from mesh file name, add multiple arguments for
 adjusting mesh yaw offset (For left/right flipping of same mesh part),
 mesh pitch for similar reason, and rot_r/p/y for determining joint
 axis of rotation
 rotation
 - Add white material
 - Mimic joints (i.e. arm joint proportional to arm servo gear joint)
 is work in progress

File: marty2_description/urdf/fixed.xacro (robot description, xacro)
@@ -1,5 +1,5 @@
 <?xml version="1.0"?>
 <robot xmlns:xacro="http://www.ros.org/wiki/xacro">
-  <xacro:macro name="fixed" params="name parent material *origin">
+  <xacro:macro name="fixed" params="name parent material mesh mesh_pitch:=0 mesh_yaw:=0 *origin">
     <joint name="${name}_joint" type="fixed">
       <xacro:insert_block name="origin"/>
@@ -15,14 +15,14 @@
       <visual>
         <geometry>
-          <mesh filename="http://0.0.0.0:8000/${name}.stl"/>
+          <mesh filename="http://0.0.0.0:8000/${mesh}.stl"/>
         </geometry>
-        <origin rpy="0 0 0" xyz="0 0 0"/>
+        <origin xyz="0 0 0" rpy="0 ${mesh_pitch} ${mesh_yaw}"/>
         <material name="${material}"/>
       </visual>
       <collision>
         <geometry>
-          <mesh filename="http://0.0.0.0:8000/${name}.stl"/>
+          <mesh filename="http://0.0.0.0:8000/${mesh}.stl"/>
         </geometry>
-        <origin rpy="0 0 0" xyz="0 0 0"/>
+        <origin xyz="0 0 0" rpy="0 ${mesh_pitch} ${mesh_yaw}"/>
         <material name="${material}"/>
       </collision>

File: marty2_description/urdf/marty2/marty2_structure.xacro (robot description, xacro)
@@ -3,8 +3,50 @@
   <xacro:include filename="$(find marty2_description)/urdf/fixed.xacro"/>
   <xacro:include filename="$(find marty2_description)/urdf/materials.xacro"/>
+  <xacro:include filename="$(find marty2_description)/urdf/revolute.xacro"/>
   <link name="base_link"/>
   <!-- Main Structure -->
-  <xacro:fixed name="martyV2-head" parent="base_link" material="blue">
+  <xacro:fixed name="head" parent="base_link" material="blue" mesh="head">
     <origin xyz="0 0 0" rpy="0 0 0"/>
   </xacro:fixed>
+  <xacro:fixed name="side_panel_left" parent="head" material="yellow" mesh="side_panel">
+    <origin xyz="0.0025 0.05744  0.04221" rpy="-0.0361 0 0"/>
+  </xacro:fixed>
+  <xacro:fixed name="side_panel_right" parent="head" material="yellow" mesh="side_panel" mesh_yaw="3.1416">
+    <origin xyz="0.0025 -0.05744 0.04221" rpy="0.0361 0 0"/>
+  </xacro:fixed>
+  <!-- Eyes -->
+  <xacro:revolute name="eye_left" parent="head" material="white" mesh="eye_left" rot_r="1">
+    <origin xyz="0.04570 0.02410 0.04671" rpy="0 0 0"/>
+  </xacro:revolute>
+  <xacro:revolute name="eye_right" parent="head" material="white" mesh="eye_right" rot_r="1">
+    <origin xyz="0.04570 -0.02410 0.04671" rpy="0 0 0"/>
+  </xacro:revolute>
+  <!-- Arms -->
+  <xacro:revolute name="arm_servo_gear_left" parent="side_panel_left" material="yellow" mesh_pitch="-0.5585" mesh="arm_servo_gear" rot_p="1">
+    <origin xyz="0 0.00025 0" rpy="0 0 0"/>
+    <!-- <mimic joint="arm_servo_gear_left_joint" multiplier="0"/> -->
+  </xacro:revolute>
+  <xacro:revolute name="arm_servo_gear_right" parent="side_panel_right" material="yellow" mesh="arm_servo_gear" mesh_pitch="-0.5585" mesh_yaw="3.1416" rot_p="1">
+    <origin xyz="0 -0.00025 0" rpy="0 0 0"/>
+    <!-- <mimic joint="arm_servo_gear_right_joint" multiplier="0"/> -->
+  </xacro:revolute>
+  <xacro:revolute name="arm_left" parent="side_panel_left" material="yellow" mesh="arm" rot_p="1">
+    <origin xyz="0 0 -0.03020" rpy="0 0 0"/>
+  </xacro:revolute>
+  <xacro:fixed name="hand_left" parent="arm_left" material="yellow" mesh="hand">
+    <origin xyz="0.00000 0.0330 -0.05539" rpy="0.3490658504 0 0"/>
+  </xacro:fixed>
+  <xacro:revolute name="arm_right" parent="side_panel_right" material="yellow" mesh="arm" mesh_yaw="3.1416" rot_p="1">
+    <origin xyz="0 0 -0.03020" rpy="0 0 0"/>
+  </xacro:revolute>
+  <xacro:fixed name="hand_right" parent="arm_right" material="yellow" mesh="hand">
+    <origin xyz="0.00000 -0.0330 -0.05539" rpy="-0.3490658504 0 0"/>
+  </xacro:fixed>
+  <!-- Legs -->
+  <xacro:fixed name="hip_left" parent="head" material="blue" mesh="hip">
+    <origin xyz="0.01087 0.04709 -0.01465" rpy="0.0000 0.0000 0.0000"/>
+  </xacro:fixed>
+  <xacro:fixed name="hip_right" parent="head" material="blue" mesh="hip">
+    <origin xyz="0.01087 -0.00941 -0.01465" rpy="0.0000 0.0000 0.0000"/>
+  </xacro:fixed>
 </robot>

File: marty2_description/urdf/materials.xacro (robot description, xacro)
@@ -7,3 +7,6 @@
     <color rgba=".8 .8 0 1"/>
   </material>
+  <material name="white">
+    <color rgba="1 1 1 1"/>
+  </material>
 </robot>

File: marty2_description/urdf/revolute.xacro (robot description, xacro)
@@ -1,9 +1,11 @@
 <?xml version="1.0"?>
 <robot xmlns:xacro="http://www.ros.org/wiki/xacro">
-  <xacro:macro name="revolute" params="name parent material *origin">
+  <xacro:macro name="revolute" params="name parent material mesh mesh_pitch:=0 mesh_yaw:=0 rot_r:=0 rot_p:=0 rot_y:=0 *origin">
     <joint name="${name}_joint" type="revolute">
       <xacro:insert_block name="origin"/>
       <parent link="${parent}"/>
       <child link="${name}"/>
+      <axis xyz="${rot_r} ${rot_p} ${rot_y}"/>
+      <limit effort="30" velocity="1.0" lower="-1.0" upper="1.0" />
     </joint>
     <link name="${name}">
@@ -15,14 +17,14 @@
       <visual>
         <geometry>
-          <mesh filename="http://0.0.0.0:8000/${name}.stl"/>
+          <mesh filename="http://0.0.0.0:8000/${mesh}.stl"/>
         </geometry>
-        <origin rpy="0 0 0" xyz="0 0 0"/>
+        <origin xyz="0 0 0" rpy="0 ${mesh_pitch} ${mesh_yaw}"/>
         <material name="${material}"/>
       </visual>
       <collision>
         <geometry>
-          <mesh filename="http://0.0.0.0:8000/${name}.stl"/>
+          <mesh filename="http://0.0.0.0:8000/${mesh}.stl"/>
         </geometry>
-        <origin rpy="0 0 0" xyz="0 0 0"/>
+        <origin xyz="0 0 0" rpy="0 ${mesh_pitch} ${mesh_yaw}"/>
         <material name="${material}"/>
       </collision>

Commit message: Update mesh filename paths to point to pkg
 - This is ROS2 friendly but requires marty2_description pkg to be
 compiled, installed and sourced locally

File: marty2_description/urdf/fixed.xacro (robot description, xacro)
@@ -15,5 +15,5 @@
       <visual>
         <geometry>
-          <mesh filename="http://0.0.0.0:8000/${mesh}.stl"/>
+          <mesh filename="package://marty2_description/meshes/${mesh}.stl"/>
         </geometry>
         <origin xyz="0 0 0" rpy="0 ${mesh_pitch} ${mesh_yaw}"/>
@@ -22,5 +22,5 @@
       <collision>
         <geometry>
-          <mesh filename="http://0.0.0.0:8000/${mesh}.stl"/>
+          <mesh filename="package://marty2_description/meshes/${mesh}.stl"/>
         </geometry>
         <origin xyz="0 0 0" rpy="0 ${mesh_pitch} ${mesh_yaw}"/>

File: marty2_description/urdf/revolute.xacro (robot description, xacro)
@@ -23,5 +23,5 @@
       <visual>
         <geometry>
-          <mesh filename="http://0.0.0.0:8000/${mesh}.stl"/>
+          <mesh filename="package://marty2_description/meshes/${mesh}.stl"/>
         </geometry>
         <origin xyz="${mesh_x} ${mesh_y} 0" rpy="${mesh_roll} ${mesh_pitch} ${mesh_yaw}"/>
@@ -30,5 +30,5 @@
       <collision>
         <geometry>
-          <mesh filename="http://0.0.0.0:8000/${mesh}.stl"/>
+          <mesh filename="package://marty2_description/meshes/${mesh}.stl"/>
         </geometry>
         <origin xyz="${mesh_x} ${mesh_y} 0" rpy="${mesh_roll} ${mesh_pitch} ${mesh_yaw}"/>
