Commit message: Simplify joint names by de-coupling from link name

File: marty2_description/ros2_control/marty2.ros2_control.xacro (robot description, xacro)
@@ -33,5 +33,5 @@
         <state_interface name="position"/>
       </joint>
-      <joint name="leg_left_thigh_front_joint">
+      <joint name="leg_left_thigh_joint">
         <command_interface name="position">
           <param name="min">-1</param>
@@ -40,5 +40,5 @@
         <state_interface name="position"/>
       </joint>
-      <joint name="leg_right_thigh_front_joint">
+      <joint name="leg_right_thigh_joint">
         <command_interface name="position">
           <param name="min">-1</param>
@@ -47,5 +47,5 @@
         <state_interface name="position"/>
       </joint>
-      <joint name="leg_left_twist_lower_joint">
+      <joint name="leg_left_twist_joint">
         <command_interface name="position">
           <param name="min">-1</param>
@@ -54,5 +54,5 @@
         <state_interface name="position"/>
       </joint>
-      <joint name="leg_right_twist_lower_joint">
+      <joint name="leg_right_twist_joint">
         <command_interface name="position">
           <param name="min">-1</param>
@@ -61,5 +61,5 @@
         <state_interface name="position"/>
       </joint>
-      <joint name="leg_left_shin_exterior_joint">
+      <joint name="leg_left_shin_joint">
         <command_interface name="position">
           <param name="min">-1</param>
@@ -68,5 +68,5 @@
         <state_interface name="position"/>
       </joint>
-      <joint name="leg_right_shin_interior_joint">
+      <joint name="leg_right_shin_joint">
         <command_interface name="position">
           <param name="min">-1</param>

File: marty2_description/urdf/marty2/marty2_structure.xacro (robot description, xacro)
@@ -52,13 +52,13 @@
     <origin xyz="0.01087 0.04709 -0.01465" rpy="0.0000 0.0000 0.0000"/>
   </xacro:fixed>
-  <xacro:revolute name="leg_left_thigh_front" parent="hip_left" material="blue" mesh="thigh" rot_p="1">
+  <xacro:revolute name="leg_left_thigh_front" parent="hip_left"  material="blue" joint_name="leg_left_thigh_joint" mesh="thigh" rot_p="1">
     <origin xyz="0.00000  0.00025 0.00000" rpy="0.0000 0.0000 0.0000"/>
     <limit effort="30" velocity="6.29" lower="-1.0" upper="1.0" />
   </xacro:revolute>
-  <xacro:revolute name="leg_left_thigh_back" parent="hip_left" material="blue" mesh="thigh" mesh_yaw="3.1416" mimic_joint="leg_left_thigh_front_joint" mimic_mult="1" rot_p="1">
+  <xacro:revolute name="leg_left_thigh_back" parent="hip_left" material="blue" mesh="thigh" mesh_yaw="3.1416" mimic_joint="leg_left_thigh_joint" mimic_mult="1" rot_p="1">
     <origin xyz="-0.01620 -0.03795  0.00000" rpy="0.0000 0.0000 0.0000"/>
     <limit effort="30" velocity="6.29" lower="-1.0" upper="1.0" />
   </xacro:revolute>
-  <xacro:revolute name="leg_left_knee_upper" parent="leg_left_thigh_front" material="blue" mesh="knee_upper" mimic_joint="leg_left_thigh_front_joint" mimic_mult="-1" rot_p="1">
+  <xacro:revolute name="leg_left_knee_upper" parent="leg_left_thigh_front" material="blue" mesh="knee_upper" mimic_joint="leg_left_thigh_joint" mimic_mult="-1" rot_p="1">
     <origin xyz="0.00000  -0.00015  -0.05000" rpy="0.0000 0.0000 0.0000"/>
     <limit effort="30" velocity="6.29" lower="-1.0" upper="1.0" />
@@ -67,5 +67,5 @@
     <origin xyz="-0.00810 -0.01885  -0.00968" rpy="0.0000 0.0000 0.0000"/>
   </xacro:fixed>
-  <xacro:revolute name="leg_left_twist_lower" parent="leg_left_twist_upper" material="yellow" mesh="twist_lower" rot_y="1">
+  <xacro:revolute name="leg_left_twist_lower" parent="leg_left_twist_upper" material="yellow" joint_name="leg_left_twist_joint" mesh="twist_lower" rot_y="1">
     <origin xyz="0.0000 0.0000 0.0000" rpy="0.0000 0.0000 0.0000"/>
     <limit effort="30" velocity="6.29" lower="-1.0" upper="1.0" />
@@ -74,13 +74,13 @@
     <origin xyz="-0.01885 0.00810 -0.02075" rpy="0.0000 0.0000 0.0000"/>
   </xacro:fixed>
-  <xacro:revolute name="leg_left_shin_exterior" parent="leg_left_knee_lower" material="blue" mesh="shin" rot_r="1">
+  <xacro:revolute name="leg_left_shin_exterior" parent="leg_left_knee_lower" material="blue" joint_name="leg_left_shin_joint" mesh="shin" rot_r="1">
     <origin xyz="0.0000 0.0000 0.0000" rpy="0.0000 0.0000 0.0000"/>
     <limit effort="30" velocity="6.29" lower="-1.0" upper="1.0" />
   </xacro:revolute>
-  <xacro:revolute name="leg_left_shin_interior" parent="leg_left_knee_lower" material="blue" mesh="shin" mesh_yaw="3.1416" mimic_joint="leg_left_shin_exterior_joint" mimic_mult="1" rot_r="1">
+  <xacro:revolute name="leg_left_shin_interior" parent="leg_left_knee_lower" material="blue" mesh="shin" mesh_yaw="3.1416" mimic_joint="leg_left_shin_joint" mimic_mult="1" rot_r="1">
     <origin xyz="0.03770  -0.01620  0.00000" rpy="0.0000 0.0000 0.0000"/>
     <limit effort="30" velocity="6.29" lower="-1.0" upper="1.0" />
   </xacro:revolute>
-  <xacro:revolute name="foot_left" parent="leg_left_shin_exterior" material="yellow" mesh="foot" mimic_joint="leg_left_shin_exterior_joint" mimic_mult="-1" rot_r="1">
+  <xacro:revolute name="foot_left" parent="leg_left_shin_exterior" material="yellow" mesh="foot" mimic_joint="leg_left_shin_joint" mimic_mult="-1" rot_r="1">
     <origin xyz="0.00000  0.00000 -0.05000" rpy="0.0000 0.0000 0.0000"/>
     <limit effort="30" velocity="6.29" lower="-1.0" upper="1.0" />
@@ -90,13 +90,13 @@
     <origin xyz="0.01087 -0.00941 -0.01465" rpy="0.0000 0.0000 0.0000"/>
   </xacro:fixed>
-  <xacro:revolute name="leg_right_thigh_front" parent="hip_right" material="blue" mesh="thigh" rot_p="1">
+  <xacro:revolute name="leg_right_thigh_front" parent="hip_right" material="blue" joint_name="leg_right_thigh_joint" mesh="thigh" rot_p="1">
     <origin xyz="0.00000  0.00025 0.00000" rpy="0.0000 0.0000 0.0000"/>
     <limit effort="30" velocity="6.29" lower="-1.0" upper="1.0" />
   </xacro:revolute>
-  <xacro:revolute name="leg_right_thigh_back" parent="hip_right" material="blue" mesh="thigh" mesh_yaw="3.1416" mimic_joint="leg_right_thigh_front_joint" mimic_mult="1" rot_p="1">
+  <xacro:revolute name="leg_right_thigh_back" parent="hip_right" material="blue" mesh="thigh" mesh_yaw="3.1416" mimic_joint="leg_right_thigh_joint" mimic_mult="1" rot_p="1">
     <origin xyz="-0.01620 -0.03795  0.00000" rpy="0.0000 0.0000 0.0000"/>
     <limit effort="30" velocity="6.29" lower="-1.0" upper="1.0" />
   </xacro:revolute>
-  <xacro:revolute name="leg_right_knee_upper" parent="leg_right_thigh_front" material="blue" mesh="knee_upper" mimic_joint="leg_right_thigh_front_joint" mimic_mult="-1" rot_p="1">
+  <xacro:revolute name="leg_right_knee_upper" parent="leg_right_thigh_front" material="blue" mesh="knee_upper" mimic_joint="leg_right_thigh_joint" mimic_mult="-1" rot_p="1">
     <origin xyz="0.00000  -0.00015  -0.05000" rpy="0.0000 0.0000 0.0000"/>
     <limit effort="30" velocity="6.29" lower="-1.0" upper="1.0" />
@@ -105,5 +105,5 @@
     <origin xyz="-0.00810 -0.01885  -0.00968" rpy="0.0000 0.0000 0.0000"/>
   </xacro:fixed>
-  <xacro:revolute name="leg_right_twist_lower" parent="leg_right_twist_upper" material="yellow" mesh="twist_lower" rot_y="1">
+  <xacro:revolute name="leg_right_twist_lower" parent="leg_right_twist_upper" material="yellow" joint_name="leg_right_twist_joint" mesh="twist_lower" rot_y="1">
     <origin xyz="0.0000 0.0000 0.0000" rpy="0.0000 0.0000 0.0000"/>
     <limit effort="30" velocity="6.29" lower="-1.0" upper="1.0" />
@@ -112,13 +112,13 @@
     <origin xyz="-0.01885 0.00810 -0.02075" rpy="0.0000 0.0000 0.0000"/>
   </xacro:fixed>
-  <xacro:revolute name="leg_right_shin_exterior" parent="leg_right_knee_lower" material="blue" mesh="shin" mesh_yaw="3.1416" mimic_joint="leg_right_shin_interior_joint" mimic_mult="1" rot_r="1">
+  <xacro:revolute name="leg_right_shin_exterior" parent="leg_right_knee_lower" material="blue" mesh="shin" mesh_yaw="3.1416" mimic_joint="leg_right_shin_joint" mimic_mult="1" rot_r="1">
     <origin xyz="0.03770  -0.01620  0.00000" rpy="0.0000 0.0000 0.0000"/>
     <limit effort="30" velocity="6.29" lower="-1.0" upper="1.0" />
   </xacro:revolute>
-  <xacro:revolute name="leg_right_shin_interior" parent="leg_right_knee_lower" material="blue" mesh="shin" rot_r="1">
+  <xacro:revolute name="leg_right_shin_interior" parent="leg_right_knee_lower" material="blue" joint_name="leg_right_shin_joint" mesh="shin" rot_r="1">
     <origin xyz="0.0000 0.0000 0.0000" rpy="0.0000 0.0000 0.0000"/>
     <limit effort="30" velocity="6.29" lower="-1.0" upper="1.0" />
   </xacro:revolute>
-  <xacro:revolute name="foot_right" parent="leg_right_shin_interior" material="yellow" mesh="foot" mesh_x="0.03790" mesh_y="-0.01620" mesh_yaw="3.1416" mimic_joint="leg_right_shin_interior_joint" mimic_mult="-1" rot_r="1">
+  <xacro:revolute name="foot_right" parent="leg_right_shin_interior" material="yellow" mesh="foot" mesh_x="0.03790" mesh_y="-0.01620" mesh_yaw="3.1416" mimic_joint="leg_right_shin_joint" mimic_mult="-1" rot_r="1">
     <origin xyz="0 0 -0.05000" rpy="0.0000 0.0000 0.0000"/>
     <limit effort="30" velocity="6.29" lower="-1.0" upper="1.0" />

File: marty2_description/urdf/revolute.xacro (robot description, xacro)
@@ -1,6 +1,9 @@
 <?xml version="1.0"?>
 <robot xmlns:xacro="http://www.ros.org/wiki/xacro">
-  <xacro:macro name="revolute" params="name parent material mesh mesh_x:=0 mesh_y:=0 mesh_roll:=0 mesh_pitch:=0 mesh_yaw:=0 rot_r:=0 rot_p:=0 rot_y:=0 mimic_joint:='' mimic_mult:='' *origin *limit">
-    <joint name="${name}_joint" type="revolute">
+  <xacro:macro name="revolute" params="name parent material joint_name:='' mesh mesh_x:=0 mesh_y:=0 mesh_roll:=0 mesh_pitch:=0 mesh_yaw:=0 rot_r:=0 rot_p:=0 rot_y:=0 mimic_joint:='' mimic_mult:='' *origin *limit">
+  <xacro:if value="${joint_name == ''}">
+    <xacro:property name="joint_name" value="${name}_joint"/>
+  </xacro:if>
+    <joint name="${joint_name}" type="revolute">
       <xacro:insert_block name="origin"/>
       <parent link="${parent}"/>

Commit message: Clean-up marty2_description with pre-commit

File: marty2_description/ros2_control/marty2.ros2_control.xacro (robot description, xacro)
@@ -6,5 +6,5 @@
         <plugin>mock_components/GenericSystem</plugin>
         <param name="calculate_dynamics">false</param>
-        <param name="custom_interface_with_following_offset"></param>
+        <param name="custom_interface_with_following_offset"/>
         <param name="disable_commands">false</param>
         <param name="mock_gpio_commands">false</param>

File: marty2_description/urdf/marty2/marty2.xacro (robot description, xacro)
@@ -7,5 +7,5 @@
   <!-- Bolt-on sensors go here -->
   <!-- <xacro:include filename="$(find marty2_description)/urdf/marty2/marty2_sensors.xacro"/> -->
-  <xacro:include filename="$(find marty2_description)/ros2_control/marty2.ros2_control.xacro" />
+  <xacro:include filename="$(find marty2_description)/ros2_control/marty2.ros2_control.xacro"/>
   <xacro:marty2_ros2_control name="marty2"/>
 </robot>

File: marty2_description/urdf/marty2/marty2_structure.xacro (robot description, xacro)
@@ -18,18 +18,18 @@
   <xacro:revolute name="eye_left" parent="head" material="white" mesh="eye_left" rot_r="1">
     <origin xyz="0.04570 0.02410 0.04671" rpy="0 0 0"/>
-    <limit effort="30" velocity="6.29" lower="-3.0" upper="0.25" />
+    <limit effort="30" velocity="6.29" lower="-3.0" upper="0.25"/>
   </xacro:revolute>
   <xacro:revolute name="eye_right" parent="head" material="white" mesh="eye_right" mesh_roll="0.01" rot_r="1" mimic_joint="eye_left_joint" mimic_mult="-1">
     <origin xyz="0.04570 -0.02410 0.04671" rpy="0 0 0"/>
-    <limit effort="30" velocity="6.29" lower="-0.25" upper="3.0" />
+    <limit effort="30" velocity="6.29" lower="-0.25" upper="3.0"/>
   </xacro:revolute>
   <!-- Left arm -->
   <xacro:revolute name="arm_servo_gear_left" parent="side_panel_left" material="yellow" mesh_pitch="-0.5585" mesh="arm_servo_gear" rot_p="1">
     <origin xyz="0 0.00025 0" rpy="0 0 0"/>
-    <limit effort="30" velocity="6.29" lower="-0.95" upper="2.05" />
+    <limit effort="30" velocity="6.29" lower="-0.95" upper="2.05"/>
   </xacro:revolute>
   <xacro:revolute name="arm_left" parent="side_panel_left" material="yellow" mesh="arm" rot_p="1" mimic_joint="arm_servo_gear_left_joint" mimic_mult="-1.307692308">
     <origin xyz="0 0 -0.03020" rpy="0 0 0"/>
-    <limit effort="30" velocity="6.29" lower="-2.68" upper="1.24" />
+    <limit effort="30" velocity="6.29" lower="-2.68" upper="1.24"/>
   </xacro:revolute>
   <xacro:fixed name="hand_left" parent="arm_left" material="yellow" mesh="hand">
@@ -39,9 +39,9 @@
   <xacro:revolute name="arm_servo_gear_right" parent="side_panel_right" material="yellow" mesh="arm_servo_gear" mesh_pitch="0.5585" mesh_yaw="3.1416" rot_p="1">
     <origin xyz="0 -0.00025 0" rpy="0 0 0"/>
-    <limit effort="30" velocity="6.29" lower="-0.95" upper="2.05" />
+    <limit effort="30" velocity="6.29" lower="-0.95" upper="2.05"/>
   </xacro:revolute>
   <xacro:revolute name="arm_right" parent="side_panel_right" material="yellow" mesh="arm" mesh_yaw="3.1416" rot_p="1" mimic_joint="arm_servo_gear_right_joint" mimic_mult="-1.307692308">
     <origin xyz="0 0 -0.03020" rpy="0 0 0"/>
-    <limit effort="30" velocity="6.29" lower="-2.68" upper="1.24" />
+    <limit effort="30" velocity="6.29" lower="-2.68" upper="1.24"/>
   </xacro:revolute>
   <xacro:fixed name="hand_right" parent="arm_right" material="yellow" mesh="hand">
@@ -52,15 +52,15 @@
     <origin xyz="0.01087 0.04709 -0.01465" rpy="0.0000 0.0000 0.0000"/>
   </xacro:fixed>
-  <xacro:revolute name="leg_left_thigh_front" parent="hip_left"  material="blue" joint_name="leg_left_thigh_joint" mesh="thigh" rot_p="1">
+  <xacro:revolute name="leg_left_thigh_front" parent="hip_left" material="blue" joint_name="leg_left_thigh_joint" mesh="thigh" rot_p="1">
     <origin xyz="0.00000  0.00025 0.00000" rpy="0.0000 0.0000 0.0000"/>
-    <limit effort="30" velocity="6.29" lower="-1.0" upper="1.0" />
+    <limit effort="30" velocity="6.29" lower="-1.0" upper="1.0"/>
   </xacro:revolute>
   <xacro:revolute name="leg_left_thigh_back" parent="hip_left" material="blue" mesh="thigh" mesh_yaw="3.1416" mimic_joint="leg_left_thigh_joint" mimic_mult="1" rot_p="1">
     <origin xyz="-0.01620 -0.03795  0.00000" rpy="0.0000 0.0000 0.0000"/>
-    <limit effort="30" velocity="6.29" lower="-1.0" upper="1.0" />
+    <limit effort="30" velocity="6.29" lower="-1.0" upper="1.0"/>
   </xacro:revolute>
   <xacro:revolute name="leg_left_knee_upper" parent="leg_left_thigh_front" material="blue" mesh="knee_upper" mimic_joint="leg_left_thigh_joint" mimic_mult="-1" rot_p="1">
     <origin xyz="0.00000  -0.00015  -0.05000" rpy="0.0000 0.0000 0.0000"/>
-    <limit effort="30" velocity="6.29" lower="-1.0" upper="1.0" />
+    <limit effort="30" velocity="6.29" lower="-1.0" upper="1.0"/>
   </xacro:revolute>
   <xacro:fixed name="leg_left_twist_upper" parent="leg_left_knee_upper" material="yellow" mesh="twist_upper">
@@ -69,5 +69,5 @@
   <xacro:revolute name="leg_left_twist_lower" parent="leg_left_twist_upper" material="yellow" joint_name="leg_left_twist_joint" mesh="twist_lower" rot_y="1">
     <origin xyz="0.0000 0.0000 0.0000" rpy="0.0000 0.0000 0.0000"/>
-    <limit effort="30" velocity="6.29" lower="-1.0" upper="1.0" />
+    <limit effort="30" velocity="6.29" lower="-1.0" upper="1.0"/>
   </xacro:revolute>
   <xacro:fixed name="leg_left_knee_lower" parent="leg_left_twist_lower" material="blue" mesh="knee_lower">
@@ -76,13 +76,13 @@
   <xacro:revolute name="leg_left_shin_exterior" parent="leg_left_knee_lower" material="blue" joint_name="leg_left_shin_joint" mesh="shin" rot_r="1">
     <origin xyz="0.0000 0.0000 0.0000" rpy="0.0000 0.0000 0.0000"/>
-    <limit effort="30" velocity="6.29" lower="-1.0" upper="1.0" />
+    <limit effort="30" velocity="6.29" lower="-1.0" upper="1.0"/>
   </xacro:revolute>
   <xacro:revolute name="leg_left_shin_interior" parent="leg_left_knee_lower" material="blue" mesh="shin" mesh_yaw="3.1416" mimic_joint="leg_left_shin_joint" mimic_mult="1" rot_r="1">
     <origin xyz="0.03770  -0.01620  0.00000" rpy="0.0000 0.0000 0.0000"/>
-    <limit effort="30" velocity="6.29" lower="-1.0" upper="1.0" />
+    <limit effort="30" velocity="6.29" lower="-1.0" upper="1.0"/>
   </xacro:revolute>
   <xacro:revolute name="foot_left" parent="leg_left_shin_exterior" material="yellow" mesh="foot" mimic_joint="leg_left_shin_joint" mimic_mult="-1" rot_r="1">
     <origin xyz="0.00000  0.00000 -0.05000" rpy="0.0000 0.0000 0.0000"/>
-    <limit effort="30" velocity="6.29" lower="-1.0" upper="1.0" />
+    <limit effort="30" velocity="6.29" lower="-1.0" upper="1.0"/>
   </xacro:revolute>
   <!-- Right leg -->
@@ -92,13 +92,13 @@
   <xacro:revolute name="leg_right_thigh_front" parent="hip_right" material="blue" joint_name="leg_right_thigh_joint" mesh="thigh" rot_p="1">
     <origin xyz="0.00000  0.00025 0.00000" rpy="0.0000 0.0000 0.0000"/>
-    <limit effort="30" velocity="6.29" lower="-1.0" upper="1.0" />
+    <limit effort="30" velocity="6.29" lower="-1.0" upper="1.0"/>
   </xacro:revolute>
   <xacro:revolute name="leg_right_thigh_back" parent="hip_right" material="blue" mesh="thigh" mesh_yaw="3.1416" mimic_joint="leg_right_thigh_joint" mimic_mult="1" rot_p="1">
     <origin xyz="-0.01620 -0.03795  0.00000" rpy="0.0000 0.0000 0.0000"/>
-    <limit effort="30" velocity="6.29" lower="-1.0" upper="1.0" />
+    <limit effort="30" velocity="6.29" lower="-1.0" upper="1.0"/>
   </xacro:revolute>
   <xacro:revolute name="leg_right_knee_upper" parent="leg_right_thigh_front" material="blue" mesh="knee_upper" mimic_joint="leg_right_thigh_joint" mimic_mult="-1" rot_p="1">
     <origin xyz="0.00000  -0.00015  -0.05000" rpy="0.0000 0.0000 0.0000"/>
-    <limit effort="30" velocity="6.29" lower="-1.0" upper="1.0" />
+    <limit effort="30" velocity="6.29" lower="-1.0" upper="1.0"/>
   </xacro:revolute>
   <xacro:fixed name="leg_right_twist_upper" parent="leg_right_knee_upper" material="yellow" mesh="twist_upper">
@@ -107,5 +107,5 @@
   <xacro:revolute name="leg_right_twist_lower" parent="leg_right_twist_upper" material="yellow" joint_name="leg_right_twist_joint" mesh="twist_lower" rot_y="1">
     <origin xyz="0.0000 0.0000 0.0000" rpy="0.0000 0.0000 0.0000"/>
-    <limit effort="30" velocity="6.29" lower="-1.0" upper="1.0" />
+    <limit effort="30" velocity="6.29" lower="-1.0" upper="1.0"/>
   </xacro:revolute>
   <xacro:fixed name="leg_right_knee_lower" parent="leg_right_twist_lower" material="blue" mesh="knee_lower">
@@ -114,13 +114,24 @@
   <xacro:revolute name="leg_right_shin_exterior" parent="leg_right_knee_lower" material="blue" mesh="shin" mesh_yaw="3.1416" mimic_joint="leg_right_shin_joint" mimic_mult="1" rot_r="1">
     <origin xyz="0.03770  -0.01620  0.00000" rpy="0.0000 0.0000 0.0000"/>
-    <limit effort="30" velocity="6.29" lower="-1.0" upper="1.0" />
+    <limit effort="30" velocity="6.29" lower="-1.0" upper="1.0"/>
   </xacro:revolute>
   <xacro:revolute name="leg_right_shin_interior" parent="leg_right_knee_lower" material="blue" joint_name="leg_right_shin_joint" mesh="shin" rot_r="1">
     <origin xyz="0.0000 0.0000 0.0000" rpy="0.0000 0.0000 0.0000"/>
-    <limit effort="30" velocity="6.29" lower="-1.0" upper="1.0" />
+    <limit effort="30" velocity="6.29" lower="-1.0" upper="1.0"/>
   </xacro:revolute>
-  <xacro:revolute name="foot_right" parent="leg_right_shin_interior" material="yellow" mesh="foot" mesh_x="0.03790" mesh_y="-0.01620" mesh_yaw="3.1416" mimic_joint="leg_right_shin_joint" mimic_mult="-1" rot_r="1">
+  <xacro:revolute
+    name="foot_right"
+    parent="leg_right_shin_interior"
+    material="yellow"
+    mesh="foot"
+    mesh_x="0.03790"
+    mesh_y="-0.01620"
+    mesh_yaw="3.1416"
+    mimic_joint="leg_right_shin_joint"
+    mimic_mult="-1"
+    rot_r="1"
+  >
     <origin xyz="0 0 -0.05000" rpy="0.0000 0.0000 0.0000"/>
-    <limit effort="30" velocity="6.29" lower="-1.0" upper="1.0" />
+    <limit effort="30" velocity="6.29" lower="-1.0" upper="1.0"/>
   </xacro:revolute>
 </robot>

File: marty2_description/urdf/revolute.xacro (robot description, xacro)
@@ -1,8 +1,11 @@
 <?xml version="1.0"?>
 <robot xmlns:xacro="http://www.ros.org/wiki/xacro">
-  <xacro:macro name="revolute" params="name parent material joint_name:='' mesh mesh_x:=0 mesh_y:=0 mesh_roll:=0 mesh_pitch:=0 mesh_yaw:=0 rot_r:=0 rot_p:=0 rot_y:=0 mimic_joint:='' mimic_mult:='' *origin *limit">
-  <xacro:if value="${joint_name == ''}">
-    <xacro:property name="joint_name" value="${name}_joint"/>
-  </xacro:if>
+  <xacro:macro
+    name="revolute"
+    params="name parent material joint_name:='' mesh mesh_x:=0 mesh_y:=0 mesh_roll:=0 mesh_pitch:=0 mesh_yaw:=0 rot_r:=0 rot_p:=0 rot_y:=0 mimic_joint:='' mimic_mult:='' *origin *limit"
+  >
+    <xacro:if value="${joint_name == ''}">
+      <xacro:property name="joint_name" value="${name}_joint"/>
+    </xacro:if>
     <joint name="${joint_name}" type="revolute">
       <xacro:insert_block name="origin"/>
@@ -13,5 +16,5 @@
         <mimic joint="${mimic_joint}" multiplier="${mimic_mult}"/>
       </xacro:if>
-      <xacro:insert_block name="limit" />
+      <xacro:insert_block name="limit"/>
     </joint>
     <link name="${name}">
